Commit message: visual.urdf 수정: origin.urdf 파일 경로 변경 및 left_front_wheel 추가, joint 정의 수정 physics.urdf 추가: 로봇 구조 및 링크, 조인트 설정 정의

File: colcon_ws/src/ku_description/urdf/physics.urdf (robot description, URDF)
Before this commit: robot myfirst, 5 links, 4 joints
Links:
- link base_link: geometry collision cylinder length=0.6 radius=0.2; visual cylinder length=0.6 radius=0.2
- link left_front_wheel: geometry collision cylinder length=0.1 radius=0.035; visual cylinder length=0.1 radius=0.035
- link left_leg: geometry collision box size=0.6 0.1 0.2; visual box size=0.6 0.1 0.2
- link right_front_wheel: geometry collision cylinder length=0.1 radius=0.035; visual cylinder length=0.1 radius=0.035
- link right_leg: geometry collision box size=0.6 0.1 0.2; visual box size=0.6 0.1 0.2

Commit message: physics.urdf 및 visual.urdf 파일 수정: 불필요한 공백 제거 및 코드 정리 limo_model.xacro 파일 추가: 로봇 모델 정의 및 매크로 추가 physics.sdf 파일 추가: 로봇 물리적 속성 정의

File: colcon_ws/src/ku_description/urdf/physics.urdf (robot description, URDF)
Before this commit: robot myfirst, 5 links, 4 joints
Links:
- link base_link: mass None -> 10
- link left_front_wheel: mass None -> 1
- link left_leg: mass None -> 10
- link right_front_wheel: mass None -> 1
- link right_leg: mass None -> 10
